Commit message: Parte 2: pista propia, bridge corregido, RViz y análisis de error
- worlds/pista.sdf generado por tools/generar_pista.py (curvas, chicana,
  estrechamiento de 0.40 m, obstáculos y muros con colisión)
- launch: argumentos world/headless/rviz/spawn, bridge unidireccional y
  /tf con gz.msgs.Pose_V, config de RViz2
- URDF: frame óptico de la cámara y odometría ground truth para análisis
- tools: prueba de recorrido automática y análisis de error
- README con dependencias y pasos de ejecución

File: src/mi_robot_diferencial/urdf/robot.urdf.xacro (robot description, xacro)
@@ -157,9 +157,17 @@
     <origin xyz="${chasis_largo/2} 0 ${chasis_alto/2}" rpy="0 0 0"/>
   </joint>
+  <!-- Frame óptico (convención REP-103: z adelante, x derecha, y abajo).
+       Las imágenes y camera_info se publican en este frame. -->
+  <link name="camera_optical_link"/>
+  <joint name="camera_optical_joint" type="fixed">
+    <parent link="camera_link"/>
+    <child link="camera_optical_link"/>
+    <origin xyz="0 0 0" rpy="${-pi/2} 0 ${-pi/2}"/>
+  </joint>
   <gazebo reference="camera_link">
     <sensor name="camera" type="camera">
       <update_rate>30</update_rate>
       <topic>/camera/image_raw</topic>
-      <gz_frame_id>camera_link</gz_frame_id>
+      <gz_frame_id>camera_optical_link</gz_frame_id>
       <camera>
         <horizontal_fov>1.85</horizontal_fov>
@@ -199,4 +207,14 @@
       <topic>/joint_states</topic>
     </plugin>
+    <!-- Odometría "ground truth" (pose real del simulador, incluye derrape).
+         Se usa solo para el análisis de error; su TF no se puentea. -->
+    <plugin filename="gz-sim-odometry-publisher-system" name="gz::sim::systems::OdometryPublisher">
+      <odom_frame>odom</odom_frame>
+      <robot_base_frame>base_footprint</robot_base_frame>
+      <odom_topic>/ground_truth/odom</odom_topic>
+      <tf_topic>/ground_truth/tf</tf_topic>
+      <odom_publish_frequency>30</odom_publish_frequency>
+      <dimensions>2</dimensions>
+    </plugin>
     <!-- Sistema de sensores -->
     <plugin filename="gz-sim-sensors-system" name="gz::sim::systems::Sensors">
